File: Hardware/SparkFun_ESP8266_Thing.brd (EAGLE design)
At the start: 55.4 x 25.9 mm, 73 parts, among them J1 DNP, Q1 2.5A/30V, U1 ESP8266, U2 MCP73831, U3 AT25SF041-SOIC8, U4 AP2112K-3.3V, U5 DNP, U6 DNP, U7 DNP, Y1 26MHz

Commit message: Mapping new parts to equivalent devices in the SparkFun libraries.
Parts:
- E1: device esp8266-development-board:TRACE_ANTENNA_2.4GHZ_25.7MM -> SparkFun-RF:TRACE_ANTENNA_2.4GHZ_25.7MM
- U1: device esp8266-development-board:QFN32 -> SparkFun-RF:QFN32
- U3: device esp8266-development-board:SO08 -> SparkFun-DigitalIC:SO08
- U5: device esp8266-development-board:UDFN8 -> SparkFun-DigitalIC:UDFN8
- U7: device esp8266-development-board:FN-6 -> SparkFun-Sensors:FN-6
Changed lines of the file:
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@@
 <layer number="56" name="wert" color="7" fill="1" visible="no" active="no"/>
 <layer number="57" name="tCAD" color="7" fill="1" visible="no" active="no"/>
+<layer number="59" name="tCarbon" color="7" fill="1" visible="no" active="no"/>
+<layer number="60" name="bCarbon" color="7" fill="1" visible="no" active="no"/>
 <layer number="90" name="Modules" color="5" fill="1" visible="no" active="no"/>
 <layer number="91" name="Nets" color="2" fill="1" visible="no" active="no"/>
@@
 <layer number="113" name="IDFDebug" color="7" fill="1" visible="no" active="yes"/>
 <layer number="116" name="Patch_BOT" color="9" fill="4" visible="no" active="yes"/>
+<layer number="118" name="Rect_Pads" color="7" fill="1" visible="yes" active="yes"/>
 <layer number="121" name="_tsilk" color="7" fill="1" visible="no" active="yes"/>
 <layer number="122" name="_bsilk" color="7" fill="1" visible="no" active="yes"/>
@@
 <layer number="127" name="_tValues" color="7" fill="1" visible="no" active="yes"/>
 <layer number="128" name="_bValues" color="7" fill="1" visible="no" active="yes"/>
+<layer number="129" name="Mask" color="7" fill="1" visible="yes" active="yes"/>
 <layer number="131" name="tAdjust" color="7" fill="1" visible="no" active="yes"/>
 <layer number="132" name="bAdjust" color="7" fill="1" visible="no" active="yes"/>
@@
 <layer number="251" name="SMDround" color="12" fill="11" visible="no" active="no"/>
 <layer number="254" name="cooling" color="7" fill="1" visible="no" active="yes"/>
+<layer number="255" name="routoute" color="7" fill="1" visible="yes" active="yes"/>
 </layers>
 <board>
@@
 </element>
 <element name="FRAME1" library="SparkFun-Aesthetics" package="CREATIVE_COMMONS" value="FRAME-LETTER" x="-2.032" y="-18.542"/>
-<element name="U1" library="esp8266-development-board" package="QFN32" value="ESP8266" x="34.29" y="16.51" rot="R180"/>
+<element name="U1" library="SparkFun-RF" package="QFN32" value="ESP8266" x="34.29" y="16.51" rot="R180">
+<attribute name="PROD_ID" value="IC-12452" x="34.29" y="16.51" size="1.778" layer="27" rot="R180" display="off"/>
+</element>
 <element name="Y1" library="things" package="CRYSTAL-SMD-3.2X2.5" value="26MHz" x="31.75" y="10.16" smashed="yes">
 <attribute name="NAME" x="31.369" y="10.287" size="0.4318" layer="25"/>
@@
 <attribute name="VALUE" x="28.448" y="5.969" size="0.4064" layer="27" font="vector"/>
 </element>
-<element name="U3" library="esp8266-development-board" package="SO08" value="AT25SF041-SOIC8" x="21.59" y="17.78" rot="R270"/>
-<element name="U5" library="esp8266-development-board" package="UDFN8" value="DNP" x="20.955" y="6.35" rot="R180"/>
+<element name="U3" library="SparkFun-DigitalIC" package="SO08" value="AT25SF041-SOIC8" x="21.59" y="17.78" rot="R270">
+<attribute name="PROD_ID" value="IC-12455" x="21.59" y="17.78" size="1.778" layer="27" rot="R270" display="off"/>
+</element>
+<element name="U5" library="SparkFun-DigitalIC" package="UDFN8" value="DNP" x="20.955" y="6.35" rot="R180">
+<attribute name="PROD_ID" value="IC-12453" x="20.955" y="6.35" size="1.778" layer="27" rot="R180" display="off"/>
+</element>
 <element name="R13" library="SparkFun-Resistors" package="0603-RES" value="2.2k" x="26.67" y="7.62" smashed="yes" rot="R90">
 <attribute name="PROD_ID" value="RES-08272" x="26.67" y="7.62" size="1.778" layer="27" font="vector" ratio="15" rot="R90" display="off"/>
@@
 <element name="LOGO3" library="SparkFun-Aesthetics" package="SFE_LOGO_FLAME_.1" value="SFE_LOGO_FLAME.1_INCH" x="2.8314625" y="0.250190625"/>
 <element name="LOGO4" library="SparkFun-Aesthetics" package="OSHW-LOGO-S" value="OSHW-LOGOS" x="7.62" y="1.905"/>
-<element name="E1" library="esp8266-development-board" package="TRACE_ANTENNA_2.4GHZ_25.7MM" value="ANTENNATRACE" x="47.752" y="14.6295" rot="R270"/>
+<element name="E1" library="SparkFun-RF" package="TRACE_ANTENNA_2.4GHZ_25.7MM" value="ANTENNATRACE" x="47.752" y="14.6295" rot="R270"/>
 <element name="C3" library="SparkFun-Capacitors" package="0603-CAP" value="10pF" x="28.575" y="10.16" smashed="yes" rot="R270">
 <attribute name="PROD_ID" value="CAP-11812" x="28.575" y="10.16" size="0.086359375" layer="27" font="vector" ratio="15" rot="R270" display="off"/>
@@
 <element name="SJ3" library="SparkFun-Passives" package="PTH-JUMPER-NC_BOTTOM_NO_SILK" value="" x="35.56" y="6.35" rot="R180"/>
 <element name="LOGO5" library="SparkFun-Aesthetics" package="SFE_LOGO_NAME_.2" value="SFE_LOGO_NAME.2_INCH" x="53.34" y="1.651" rot="R90"/>
-<element name="U7" library="esp8266-development-board" package="FN-6" value="DNP" x="20.955" y="12.065" rot="R180"/>
+<element name="U7" library="SparkFun-Sensors" package="FN-6" value="DNP" x="20.955" y="12.065" rot="R180"/>
 <element name="C12" library="SparkFun-Capacitors" package="0603-CAP" value="DNP" x="24.13" y="6.35" rot="R90">
 <attribute name="PROD_ID" value="CAP-00810" x="24.13" y="6.35" size="0.8128" layer="27" font="vector" ratio="15" rot="R90" display="off"/>
